File: PCB/CobraPad/CobraPad.kicad_pcb (KiCad board)
At the start: 2 copper layers, 99 x 99 mm, 39 parts, among them SW1 SW_Push, SW2 SW_Push, SW3 SW_Push, SW4 SW_Push, SW5 SW_Push, SW6 SW_Push, SW7 SW_Push, SW8 SW_Push, SW9 RotaryEncoder_Switch, U1 MOUDLE-SEEEDUINO-XIAO, U2 ER_OLEDM0.91_1x-I2C

Commit message: Final Case
Parts:
- moved U2 4.47 mm to (79.5, 116.8)
- moved U1 1.91 mm to (96.6, 96.0)
Routing:
- net Net-(U1-GND): track 66.5 -> 84.6 mm, vias 0 -> 2
- net Net-(U1-PA8_A4_D4_SDA): track 30.7 -> 39.9 mm
- net /Col2: track 303.7 -> 308.8 mm
- net /Row2: track 171.3 -> 173.8 mm
- net Net-(D9-DIN): track 71.8 -> 74.2 mm
- net Net-(U1-PA7_A8_D8_SCK): track 11.4 -> 8.98 mm
- net Net-(U1-PA5_A9_D9_MISO): track 19.0 -> 16.6 mm
- net /Col1: track 123.7 -> 125.7 mm
- net /Col3: track 149.2 -> 151.1 mm
- net Net-(U1-3V3): track 35.0 -> 33.4 mm
- net /Col4: track 140.9 -> 142.5 mm
- net Net-(U1-PA9_A5_D5_SCL): track 29.8 -> 29.1 mm
